Commit message: gravity 90% done

File: FACTR_Teleop/src/factr_teleop/factr_teleop/urdf/factr_teleop_franka.urdf (robot description, URDF)
Before this commit: robot factr_teleop_franka, 8 links, 7 joints
Links:
- link link_4: mass 0.051 -> 0.029
- link link_5: mass 0.048 -> 0.027
- link link_6: mass 0.035 -> 0.012
- link link_7: mass 0.051 -> 0.046
Joints:
- joint joint_4: axis 0 0 1 -> 0 -1 0; limit lower=-3.0718 upper=-0.0698 effort=0.92 velocity=6.8 -> lower=-10 upper=10 effort=0.92 velocity=6.8
- joint joint_6: axis 0 0 1 -> 0 0 -1

Commit message: updated the urdf file

File: FACTR_Teleop/src/factr_teleop/factr_teleop/urdf/factr_teleop_franka.urdf (robot description, URDF)
Before this commit: robot factr_teleop_franka, 8 links, 7 joints
Links:
- link link_4: mass 0.029 -> 0.037
- link link_5: mass 0.027 -> 0.031
- link link_6: mass 0.012 -> 0.022
- link link_7: mass 0.046 -> 0.032
Joints:
- joint joint_6: axis 0 0 -1 -> 0 0 1

Commit message: small changes

File: FACTR_Teleop/src/factr_teleop/factr_teleop/urdf/factr_teleop_franka.urdf (robot description, URDF)
Before this commit: robot factr_teleop_franka, 8 links, 7 joints
Links:
- link link_1: mass 0.115 -> 0.094
- link link_2: mass 0.042 -> 0.03015
- link link_3: mass 0.113 -> 0.0938
- link link_4: mass 0.037 -> 0.0297
- link link_5: mass 0.031 -> 0.0292
- link link_6: mass 0.022 -> 0.0282
- link link_7: mass 0.032 -> 0.046
