Commit message: Checkpoint DFC-owned FACTR calibration and diagnostics

File: FACTR_Teleop/src/factr_teleop/factr_teleop/urdf/flexiv_teleop_neg45_x_lighter.urdf (robot description, URDF)
Before this commit: robot flexiv_teleop_neg45_x_lighter, 9 links, 8 joints
Links:
- removed link link_7
- added link rail_carriage_link, mass 0.214492; collision mesh filename=link_7.stl scale=0.001 0.001 0.001; visual mesh filename=link_7.stl scale=0.001 0.001 0.001
Joints:
- joint joint_7: child link_7 -> rail_carriage_link
